File: hardware/schematics/Schematic.sch (EAGLE design)
At the start: 1 part, among them IC1 MEGA8-AI

Commit message: Add files via upload
Parts:
- added BLUETOOTH_DTR: (no value), pinhead:PINHD-1X1
- added BLUETOOTH_SERIAL_PORT: (no value), pinhead:PINHD-1X2
Connections:
- new net BLUETOOTH_RX: BLUETOOTH_SERIAL_PORT.1, IC1.PD0(RXD)
- new net BLUETOOTH_TX: BLUETOOTH_SERIAL_PORT.2, IC1.PD1(TXD)
- new net RESET_SUBSYSTEM: IC1.PC6(/RESET)
- new net SPI_MISO: IC1.PB4(MISO)
- new net SPI_MOSI: IC1.PB3(MOSI/OC2)
- new net SPI_SCK: IC1.PB5(SCK)
- new net SPI_SS: IC1.PB2(SS/OC1B)
- new net VCC: IC1.VCC@1, IC1.VCC@2
Other:
- moved on the sheet: IC1
Changed lines of the file:
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@@
 <part name="SUPPLY1" library="supply2" deviceset="GND" device=""/>
 <part name="SUPPLY2" library="supply2" deviceset="GND" device=""/>
+<part name="P+1" library="supply1" deviceset="VCC" device=""/>
+<part name="BLUETOOTH_SERIAL_PORT" library="pinhead" deviceset="PINHD-1X2" device=""/>
+<part name="BLUETOOTH_DTR" library="pinhead" deviceset="PINHD-1X1" device=""/>
+<part name="FRAME1" library="frames" deviceset="A3L-LOC" device=""/>
 </parts>
 <sheets>
 <sheet>
 <plain>
+<wire x1="15.24" y1="248.92" x2="15.24" y2="200.66" width="0.1524" layer="97"/>
+<wire x1="15.24" y1="200.66" x2="88.9" y2="200.66" width="0.1524" layer="97"/>
+<wire x1="88.9" y1="200.66" x2="88.9" y2="248.92" width="0.1524" layer="97"/>
+<wire x1="88.9" y1="248.92" x2="15.24" y2="248.92" width="0.1524" layer="97"/>
+<wire x1="15.24" y1="195.58" x2="15.24" y2="134.62" width="0.1524" layer="97"/>
+<wire x1="15.24" y1="134.62" x2="96.52" y2="134.62" width="0.1524" layer="97"/>
+<wire x1="96.52" y1="134.62" x2="96.52" y2="195.58" width="0.1524" layer="97"/>
+<wire x1="15.24" y1="195.58" x2="96.52" y2="195.58" width="0.1524" layer="97"/>
 </plain>
 <instances>
-<instance part="IC1" gate="G$1" x="10.16" y="71.12"/>
-<instance part="SUPPLY1" gate="GND" x="-22.86" y="60.96"/>
-<instance part="SUPPLY2" gate="GND" x="-22.86" y="88.9"/>
+<instance part="IC1" gate="G$1" x="180.34" y="147.32"/>
+<instance part="SUPPLY1" gate="GND" x="152.4" y="144.78"/>
+<instance part="SUPPLY2" gate="GND" x="147.32" y="170.18"/>
+<instance part="P+1" gate="VCC" x="142.24" y="142.24"/>
+<instance part="BLUETOOTH_SERIAL_PORT" gate="G$1" x="238.76" y="147.32" smashed="yes">
+<attribute name="NAME" x="219.71" y="158.115" size="1.778" layer="95"/>
+<attribute name="VALUE" x="232.41" y="142.24" size="1.778" layer="96"/>
+</instance>
+<instance part="BLUETOOTH_DTR" gate="G$1" x="48.26" y="233.68" smashed="yes" rot="R90">
+<attribute name="NAME" x="59.69" y="238.125" size="1.778" layer="95" rot="R180"/>
+<attribute name="VALUE" x="53.34" y="227.33" size="1.778" layer="96" rot="R90"/>
+</instance>
+<instance part="FRAME1" gate="G$1" x="0" y="0"/>
 </instances>
 <busses>
 </busses>
 <nets>
+<net name="VCC" class="0">
+<segment>
+<pinref part="P+1" gate="VCC" pin="VCC"/>
+<wire x1="142.24" y1="139.7" x2="142.24" y2="137.16" width="0.1524" layer="91"/>
+<pinref part="IC1" gate="G$1" pin="VCC@1"/>
+<wire x1="142.24" y1="137.16" x2="157.48" y2="137.16" width="0.1524" layer="91"/>
+<pinref part="IC1" gate="G$1" pin="VCC@2"/>
+<wire x1="157.48" y1="137.16" x2="157.48" y2="134.62" width="0.1524" layer="91"/>
+<junction x="157.48" y="137.16"/>
+</segment>
+</net>
 <net name="GND" class="0">
 <segment>
-<pinref part="IC1" gate="G$1" pin="GND"/>
-<pinref part="SUPPLY2" gate="GND" pin="GND"/>
-<wire x1="-12.7" y1="91.44" x2="-22.86" y2="91.44" width="0.1524" layer="91"/>
+<pinref part="IC1" gate="G$1" pin="GND@2"/>
+<pinref part="IC1" gate="G$1" pin="GND@1"/>
+<wire x1="157.48" y1="142.24" x2="157.48" y2="139.7" width="0.1524" layer="91"/>
+<wire x1="157.48" y1="142.24" x2="157.48" y2="147.32" width="0.1524" layer="91"/>
+<pinref part="SUPPLY1" gate="GND" pin="GND"/>
+<wire x1="157.48" y1="147.32" x2="152.4" y2="147.32" width="0.1524" layer="91"/>
+<junction x="157.48" y="142.24"/>
 </segment>
 <segment>
-<pinref part="IC1" gate="G$1" pin="GND@2"/>
-<pinref part="SUPPLY1" gate="GND" pin="GND"/>
-<wire x1="-12.7" y1="63.5" x2="-22.86" y2="63.5" width="0.1524" layer="91"/>
-<pinref part="IC1" gate="G$1" pin="GND@1"/>
-<wire x1="-12.7" y1="66.04" x2="-12.7" y2="63.5" width="0.1524" layer="91"/>
+<pinref part="IC1" gate="G$1" pin="GND"/>
+<wire x1="157.48" y1="167.64" x2="152.4" y2="167.64" width="0.1524" layer="91"/>
+<wire x1="152.4" y1="167.64" x2="152.4" y2="172.72" width="0.1524" layer="91"/>
+<pinref part="SUPPLY2" gate="GND" pin="GND"/>
+<wire x1="152.4" y1="172.72" x2="147.32" y2="172.72" width="0.1524" layer="91"/>
 </segment>
 </net>
+<net name="BLUETOOTH_RX" class="0">
+<segment>
+<pinref part="IC1" gate="G$1" pin="PD0(RXD)"/>
+<label x="210.82" y="149.86" size="1.778" layer="95"/>
+<pinref part="BLUETOOTH_SERIAL_PORT" gate="G$1" pin="1"/>
+<wire x1="205.74" y1="149.86" x2="236.22" y2="149.86" width="0.1524" layer="91"/>
+<junction x="236.22" y="149.86"/>
+</segment>
+</net>
+<net name="BLUETOOTH_TX" class="0">
+<segment>
+<pinref part="IC1" gate="G$1" pin="PD1(TXD)"/>
+<label x="210.82" y="147.32" size="1.778" layer="95"/>
+<pinref part="BLUETOOTH_SERIAL_PORT" gate="G$1" pin="2"/>
+<wire x1="205.74" y1="147.32" x2="236.22" y2="147.32" width="0.1524" layer="91"/>
+<junction x="236.22" y="147.32"/>
+</segment>
+</net>
+<net name="SPI_MISO" class="0">
+<segment>
+<pinref part="IC1" gate="G$1" pin="PB4(MISO)"/>
+<wire x1="220.98" y1="116.84" x2="205.74" y2="116.84" width="0.1524" layer="91"/>
+<label x="220.98" y="116.84" size="1.778" layer="95"/>
+</segment>
+</net>
+<net name="SPI_MOSI" class="0">
+<segment>
+<pinref part="IC1" gate="G$1" pin="PB3(MOSI/OC2)"/>
+<wire x1="205.74" y1="119.38" x2="220.98" y2="119.38" width="0.1524" layer="91"/>
+<label x="220.98" y="119.38" size="1.778" layer="95"/>
+</segment>
+</net>
+<net name="SPI_SCK" class="0">
+<segment>
+<pinref part="IC1" gate="G$1" pin="PB5(SCK)"/>
+<wire x1="205.74" y1="114.3" x2="220.98" y2="114.3" width="0.1524" layer="91"/>
+<label x="220.98" y="114.3" size="1.778" layer="95"/>
+</segment>
+</net>
+<net name="SPI_SS" class="0">
+<segment>
+<pinref part="IC1" gate="G$1" pin="PB2(SS/OC1B)"/>
+<wire x1="205.74" y1="121.92" x2="220.98" y2="121.92" width="0.1524" layer="91"/>
+<label x="220.98" y="121.92" size="1.778" layer="95"/>
+</segment>
+</net>
+<net name="RESET_SUBSYSTEM" class="0">
+<segment>
+<pinref part="IC1" gate="G$1" pin="PC6(/RESET)"/>
+<wire x1="157.48" y1="172.72" x2="154.94" y2="172.72" width="0.1524" layer="91"/>
+<wire x1="154.94" y1="172.72" x2="154.94" y2="182.88" width="0.1524" layer="91"/>
+<label x="144.78" y="182.88" size="1.778" layer="95"/>
+</segment>
+<segment>
+<wire x1="30.48" y1="213.36" x2="66.04" y2="213.36" width="0.1524" layer="91"/>
+<label x="40.64" y="208.28" size="1.778" layer="95"/>
+</segment>
+</net>

Commit message: Add files via upload
Parts:
- added C1, C2: 22p, rcl:C-EUC0603
- added C3: 1u, rcl:C-EUC0603
- added JTAG: (no value), pinhead:PINHD-2X3
- added R1: (no value), resistor:R-US_R0603
- added S1: SKHMPSE010, switch:SKHMPSE010
- added Y1: 16 mhz, SparkFun-FreqCtrl:CRYSTALHC49UV
Connections:
- removed net RESET_SUBSYSTEM: IC1.PC6(/RESET)
- new net N$1: BLUETOOTH_DTR.1, C3.1
- new net RESET_PIN: C3.2, IC1.PC6(/RESET), JTAG.5, R1.1, S1.2.1
- new net XTAL1: C2.2, IC1.PB6(XTAL1/TOSC1), Y1.2
- new net XTAL2: C1.2, IC1.PB7(XTAL2/TOSC2), Y1.1
- net GND: now also C1.1, C2.1, JTAG.6, S1.1.1
- net SPI_MISO: now also JTAG.1
- net SPI_MOSI: now also JTAG.4
- net SPI_SCK: now also JTAG.3
- net VCC: now also IC1.AREF, IC1.AVCC, JTAG.2, R1.2
Other:
- note added: "Clock Subsystem"
- note added: "JTAG"
- note added: "Reset Subsystem"
- moved on the sheet: BLUETOOTH_DTR

Commit message: schematic additions
added power schematics
Parts:
- added C10, C9: 4.7uF, SparkFun:CAP0402-CAP
- added C4: 22uF, CH_passive:CAP0805
- added C5: 0.1uF, SparkFun:CAP0402-CAP
- added C6: 10uF, CH_passive:CAP1206
- added D4: red, SparkFun:LED0603
- added IC2: MC33269D-3.3, linear:MC33269D-3.3
- added JP1: LiPo, SparkFun:M02-JST-2MM-SMT
- added JP12: LiPoIN, SparkFun:M02PTH
- added JP15, JP16: FIDUCIALUFIDUCIAL, SparkFun:FIDUCIALUFIDUCIAL
- added JP3: LOGO-SFENEW, SparkFun:LOGO-SFENEW
- added JP4: LOGO-SFESK, SparkFun:LOGO-SFESK
- added JP5, JP6, JP7, JP8: STAND-OFF, SparkFun:STAND-OFF
- added JP9: IN, SparkFun:M02PTH
- added L1: 4.7uH, 1.2A, SparkFun:INDUCTOR.
- added R5: 2k, SparkFun:RESISTOR0402-RES
- added R6: 220k, SparkFun:RESISTOR0402-RES
- added R7: 2M, SparkFun:RESISTOR0402-RES
- added R9: 470, SparkFun:RESISTOR0402-RES
- added U$1: OSHW-LOGOS, SparkFun:OSHW-LOGOS
- added U$2: CREATIVE_COMMONS, SparkFun-Aesthetics:CREATIVE_COMMONS
- added U1: MCP73831, SparkFun:MCP73831
- added U2: TPS61200, SparkFun:TPS61200
- added X1: USB-MICROB, SparkFun:USB-MICROB
Connections:
- new net 5VIN: C9.1, D4.A, JP9.1, U1.VIN, X1.VBUS
- new net FB: R6.2, R7.1, U2.FB
- new net GND1: R6.1
- new net N$11: R5.1, U1.PROG
- new net N$14: R9.1, U1.STAT
- new net N$2: L1.1, U2.L
- new net N$3: C5.1, U2.VAUX
- new net N$8: D4.C, R9.2
- new net SUPPLY_3.3V: IC2.VO
- new net SUPPLY_5V: C4.1, IC2.VI, R7.2, U2.VOUT
- new net VBATT: C10.1, C6.1, JP1.2, JP12.1, L1.2, U1.VBAT, U2.EN, U2.PS, U2.UVLO, U2.VIN
- net GND: now also C10.2, C4.2, C5.2, C6.2, C9.2, IC2.ADJ, JP1.1, JP12.2, JP9.2, R5.2, U1.VSS, U2.GND, U2.PAD@1, U2.PAD@2, U2.PAD@3, U2.PAD@4, U2.PAD@5, U2.PGND, X1.GND
Other:
- note added: "A.Weiss"
- note added: "GND1 as recommended by datasheet to separate ground for control circuit"
- note added: "LiPo Charger"
- note added: "Special Thanks to Oleg at Circuits at Home for the TPS61200 design"
- note added: "Switching Regulator"
